Commit message: Stable First COmmit

File: build/bvcc.urdf (robot description, URDF)
Before this commit: robot mintaur, 7 links, 6 joints
Links:
- link base_link: geometry collision box size=0.51 0.2 0.15; visual mesh filename=/home/eichmeierbr/mrob/src/miniProject/urdf/avc_urdf/meshes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 scale=0.15 0.15 0.15

File: urdf/bvc.xacro (robot description, xacro)
@@ -1,7 +1,7 @@
 <?xml version="1.0"?>
 <robot xmlns:xacro="http://www.ros.org/wiki/xacro" name="mintaur">
-    <xacro:include filename="/home/eichmeierbr/mrob/src/miniProject/urdf/experiment/materials.xacro" />
-	<xacro:include filename="/home/eichmeierbr/mrob/src/miniProject/urdf/experiment/properties.xacro" />
-    <xacro:include filename="/home/eichmeierbr/mrob/src/miniProject/urdf/experiment/links.xacro" />
+    <xacro:include filename="$(find avc_urdf)/urdf/materials.xacro" />
+	<xacro:include filename="$(find avc_urdf)/urdf/properties.xacro" />
+    <xacro:include filename="$(find avc_urdf)/urdf/links.xacro" />
   <xacro:base_link/>
   <xacro:wheel side="right" fob="front" sideDim="${rightWheelDist}" fobDim="${frontWheelDist}" />
@@ -10,4 +10,4 @@
   <xacro:wheel side="left" fob="back" sideDim="${leftWheelDist}" fobDim="${backWheelDist}" />
   <!-- <xacro:imu /> -->
-    <xacro:include filename="/home/eichmeierbr/mrob/src/miniProject/urdf/experiment/gazebo.xacro" />
+    <xacro:include filename="$(find avc_urdf)/urdf/gazebo.xacro" />
 </robot>

File: urdf/links.xacro (robot description, xacro)
@@ -9,5 +9,5 @@
         <visual>
             <geometry>
-                <mesh filename="/home/eichmeierbr/mrob/src/miniProject/urdf/meshes/chassis.DAE" scale="${chassisScale} ${chassisScale} ${chassisScale}"/>
+                <mesh filename="$(find avc_urdf)/meshes/chassis.DAE" scale="${chassisScale} ${chassisScale} ${chassisScale}"/>
             </geometry>
             <origin rpy="1.57 0 3.14" xyz="0 0 0" />

Commit message: Chassis and Wheel Mesh

File: build/bvcc.urdf (robot description, URDF)
Before this commit: robot mintaur, 7 links, 6 joints
Links:
- link base_link: geometry collision box size=0.51 0.2 0.15; visual mesh filename=/home/eichmeierbr/mrob/src/miniProject/urdf/avc_urdf/meshes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 scale=0.001 0.001 0.001
- link left_back_wheel: geometry collision cylinder length=0.043 radius=0.05; visual mesh filename=/home/eichmeierbr/mrob/src/miniProject/urdf/avc_urdf/meshes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 scale=0.001 0.001 0.001
- link left_front_wheel: geometry collision cylinder length=0.043 radius=0.05; visual mesh filename=/home/eichmeierbr/mrob/src/miniProject/urdf/avc_urdf/meshes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 scale=0.001 0.001 0.001
- link right_back_wheel: geometry collision cylinder length=0.043 radius=0.05; visual mesh filename=/home/eichmeierbr/mrob/src/miniProject/urdf/avc_urdf/meshes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 scale=0.001 0.001 0.001
- link right_front_wheel: geometry collision cylinder length=0.043 radius=0.05; visual mesh filename=/home/eichmeierbr/mrob/src/miniProject/urdf/avc_urdf/meshes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 scale=0.001 0.001 0.001

File: urdf/bvc.xacro (robot description, xacro)
@@ -10,4 +10,5 @@
   <xacro:wheel side="left" fob="back" sideDim="${leftWheelDist}" fobDim="${backWheelDist}" />
   <!-- <xacro:imu /> -->
+  <!-- <xacro:lidar /> TODO -->
     <xacro:include filename="$(find avc_urdf)/urdf/gazebo.xacro" />
 </robot>

File: urdf/geometries.xacro (robot description, xacro)
@@ -1,4 +1,10 @@
 <?xml version="1.0"?>
 <robot xmlns:xacro="http://www.ros.org/wiki/xacro" name="mintaur">
+    <xacro:macro name="chassis_mesh_geometry">
+        <geometry>
+            <mesh filename="$(find avc_urdf)/meshes/chassis2.DAE" scale="${chassisScale} ${chassisScale} ${chassisScale}"/>
+         </geometry>
+         <origin rpy="1.57 0 0" xyz="${chassisMeshXoffset} ${chassisMeshYoffset} ${chassisMeshZoffset}" />
+	</xacro:macro>
 	<xacro:macro name="box_geometry">
        <geometry>
@@ -11,4 +17,15 @@
         </geometry>
 	</xacro:macro> -->
+    <xacro:macro name="wheel_mesh_geometry" params="side">
+        <geometry>
+            <mesh filename="$(find avc_urdf)/meshes/wheels.DAE" scale="${wheelScale} ${wheelScale} ${wheelScale}"/>
+         </geometry>
+            <xacro:if value="${side =='right'}">
+                <origin rpy="1.57 0 0" xyz="0 ${wheelMeshYoffset} 0" />
+            </xacro:if>
+            <xacro:if value="${side =='left'}">
+                <origin rpy="1.57 0 3.14" xyz="${wheelMeshXoffset} ${wheelMeshYoffset} ${wheelMeshZoffset}" />
+            </xacro:if>
+	</xacro:macro>
     <xacro:macro name="wheel_geometry">
         <geometry>

File: urdf/joints.xacro (robot description, xacro)
@@ -34,3 +34,11 @@
         </joint>
 	</xacro:macro> -->
+    <xacro:macro name="chassis_box_joint">
+        <joint name="chassis_box_joint" type="fixed">
+            <axis xyz="0 1 0"/>
+            <parent link="base_link"/>
+            <child link="chassis_box_link"/>
+            <origin xyz="0 0 0" />
+        </joint>
+	</xacro:macro>
 </robot>

File: urdf/links.xacro (robot description, xacro)
@@ -8,10 +8,5 @@
     <link name="base_link">
         <visual>
-            <geometry>
-                <mesh filename="$(find avc_urdf)/meshes/chassis.DAE" scale="${chassisScale} ${chassisScale} ${chassisScale}"/>
-            </geometry>
-            <origin rpy="1.57 0 3.14" xyz="0 0 0" />
-            <!-- <xacro:box_geometry />
-            <material name="blue"/> -->
+            <xacro:chassis_mesh_geometry />
         </visual>
         <collision>
@@ -24,6 +19,5 @@
     <link name="${side}_${fob}_wheel">
         <visual>
-            <xacro:wheel_geometry />
-            <material name="white"/>
+            <xacro:wheel_mesh_geometry side="${side}"/>
         </visual>
         <collision>

File: urdf/properties.xacro (robot description, xacro)
@@ -13,5 +13,8 @@
     <xacro:property name="chassisIyz" value="0.4"/>
     <xacro:property name="chassisIzz" value="0.4"/>
-     <xacro:property name="chassisScale" value="0.15"/>
+     <xacro:property name="chassisScale" value="0.001"/>
+    <xacro:property name="chassisMeshXoffset" value="-0.125"/>
+    <xacro:property name="chassisMeshYoffset" value="-0.070"/>
+    <xacro:property name="chassisMeshZoffset" value="-0.085"/>
  <!-- ______________Wheel parameters__________________________ -->
     <!-- Wheel Rotation Limits> -->
@@ -24,4 +27,8 @@
     <xacro:property name="backWheelDist" value="-0.1763" />
     <xacro:property name="wheelDrop" value="-0.075" />
+    <xacro:property name="wheelScale" value="0.001"/>
+    <xacro:property name="wheelMeshXoffset" value="0"/>
+    <xacro:property name="wheelMeshYoffset" value="0.022"/>
+    <xacro:property name="wheelMeshZoffset" value="0"/>
     <!-- Wheel Physical Propreties-->
     <xacro:property name="wheelThickness" value="0.043" />

Commit message: Fixed launch files and mesh colors.

File: build/bvcc.urdf (robot description, URDF)
Before this commit: robot mintaur, 7 links, 6 joints
Links:
- link base_link: mass 10 -> 1; geometry collision box size=0.51 0.2 0.15; visual mesh filename=/home/eichmeierbr/mrob/src/avc_urdf/meshes/chassis2.DAE scale=0.001 0.001 0.001
- link left_back_wheel: mass 10 -> 1; geometry collision cylinder length=0.043 radius=0.05; visual mesh filename=/home/eichmeierbr/mrob/src/avc_urdf/meshes/wheels.DAE scale=0.001 0.001 0.001
- link left_front_wheel: mass 10 -> 1; geometry collision cylinder length=0.043 radius=0.05; visual mesh filename=/home/eichmeierbr/mrob/src/avc_urdf/meshes/wheels.DAE scale=0.001 0.001 0.001
- link right_back_wheel: mass 10 -> 1; geometry collision cylinder length=0.043 radius=0.05; visual mesh filename=/home/eichmeierbr/mrob/src/avc_urdf/meshes/wheels.DAE scale=0.001 0.001 0.001
- link right_front_wheel: mass 10 -> 1; geometry collision cylinder length=0.043 radius=0.05; visual mesh filename=/home/eichmeierbr/mrob/src/avc_urdf/meshes/wheels.DAE scale=0.001 0.001 0.001

File: urdf/gazebo.xacro (robot description, xacro)
@@ -13,5 +13,6 @@
 		<plugin name="gazebo_ros_control" filename="libgazebo_ros_control.so">
 			<robotNamespace>/</robotNamespace>
-			<!-- <robotSimType>gazebo_ros_control/DefaultRobotHWSim</robotSimType> -->
+			<robotSimType>gazebo_ros_control/DefaultRobotHWSim</robotSimType>
+            <legacyModeNS>true</legacyModeNS>
 		</plugin>
 	</gazebo>

File: urdf/geometries.xacro (robot description, xacro)
@@ -3,5 +3,5 @@
     <xacro:macro name="chassis_mesh_geometry">
         <geometry>
-            <mesh filename="$(find avc_urdf)/meshes/chassis2.DAE" scale="${chassisScale} ${chassisScale} ${chassisScale}"/>
+            <mesh filename="file:///$(find avc_urdf)/meshes/chassis2.DAE" scale="${chassisScale} ${chassisScale} ${chassisScale}"/>
          </geometry>
          <origin rpy="1.57 0 0" xyz="${chassisMeshXoffset} ${chassisMeshYoffset} ${chassisMeshZoffset}" />
@@ -19,5 +19,5 @@
     <xacro:macro name="wheel_mesh_geometry" params="side">
         <geometry>
-            <mesh filename="$(find avc_urdf)/meshes/wheels.DAE" scale="${wheelScale} ${wheelScale} ${wheelScale}"/>
+            <mesh filename="file:///$(find avc_urdf)/meshes/wheels.DAE" scale="${wheelScale} ${wheelScale} ${wheelScale}"/>
          </geometry>
             <xacro:if value="${side =='right'}">
@@ -25,5 +25,5 @@
             </xacro:if>
             <xacro:if value="${side =='left'}">
-                <origin rpy="1.57 0 3.14" xyz="${wheelMeshXoffset} ${wheelMeshYoffset} ${wheelMeshZoffset}" />
+                <origin rpy="1.57 0 3.14" xyz="${wheelMeshXoffset} ${wheelMeshYoffsetLeft} ${wheelMeshZoffset}" />
             </xacro:if>
 	</xacro:macro>

File: urdf/links.xacro (robot description, xacro)
@@ -9,4 +9,5 @@
         <visual>
             <xacro:chassis_mesh_geometry />
+            <material name="white" />
         </visual>
         <collision>
@@ -20,4 +21,5 @@
         <visual>
             <xacro:wheel_mesh_geometry side="${side}"/>
+            <material name="black" />
         </visual>
         <collision>

File: urdf/properties.xacro (robot description, xacro)
@@ -6,11 +6,11 @@
     <xacro:property name="chassisW" value="0.2" />
     <xacro:property name="chassisH" value="0.15" />
-    <xacro:property name="chassisMass" value="10"/>
+    <xacro:property name="chassisMass" value="1"/>
     <xacro:property name="chassisIxx" value="0.4"/>
     <xacro:property name="chassisIxy" value="0.4"/>
     <xacro:property name="chassisIyy" value="0.4"/>
-    <xacro:property name="chassisIxz" value="0.4"/>
-    <xacro:property name="chassisIyz" value="0.4"/>
-    <xacro:property name="chassisIzz" value="0.4"/>
+    <xacro:property name="chassisIxz" value="0.0"/>
+    <xacro:property name="chassisIyz" value="0.0"/>
+    <xacro:property name="chassisIzz" value="0.0"/>
      <xacro:property name="chassisScale" value="0.001"/>
     <xacro:property name="chassisMeshXoffset" value="-0.125"/>
@@ -30,4 +30,5 @@
     <xacro:property name="wheelMeshXoffset" value="0"/>
     <xacro:property name="wheelMeshYoffset" value="0.022"/>
+   <xacro:property name="wheelMeshYoffsetLeft" value="-0.022"/>
     <xacro:property name="wheelMeshZoffset" value="0"/>
     <!-- Wheel Physical Propreties-->
@@ -36,11 +37,11 @@
     <xacro:property name="axleEffort" value="0.001"/>
     <xacro:property name="axleVelocity" value="0.5"/>
-    <xacro:property name="wheelMass" value="10"/>
+    <xacro:property name="wheelMass" value="1"/>
     <xacro:property name="wheelIxx" value="0.4"/>
-    <xacro:property name="wheelIxy" value="0.4"/>
     <xacro:property name="wheelIyy" value="0.4"/>
-    <xacro:property name="wheelIxz" value="0.4"/>
-    <xacro:property name="wheelIyz" value="0.4"/>
     <xacro:property name="wheelIzz" value="0.4"/>
+    <xacro:property name="wheelIxy" value="0.0"/>
+    <xacro:property name="wheelIxz" value="0.0"/>
+    <xacro:property name="wheelIyz" value="0.0"/>
     <!-- Wheel Gazebo and Inertial Properties -->
     <xacro:property name="wheelMu1" value="200"/>

File: urdf/transmissions.xacro (robot description, xacro)
@@ -8,5 +8,6 @@
             </actuator>
             <joint name="base_to_${side}_${fob}_axle">
-                <hardwareInterface>PositionJointInterface</hardwareInterface>
+                <hardwareInterface>hardware_interface/PositionJointInterface</hardwareInterface>
+                <!-- <hardwareInterface>hardware_interface/PositionJointInterface</hardwareInterface> -->
             </joint>
         </transmission>

Commit message: Start of my branch for stuff not quite ready for the big stuff

File: build/bvcc.urdf (robot description, URDF)
Before this commit: robot mintaur, 7 links, 6 joints
Links:
- link base_link: geometry collision box size=0.51 0.2 0.15; visual box size=0.51 0.2 0.15
- link left_back_wheel: geometry collision cylinder length=0.043 radius=0.05; visual cylinder length=0.043 radius=0.05
- link left_front_wheel: geometry collision cylinder length=0.043 radius=0.05; visual cylinder length=0.043 radius=0.05
- link right_back_wheel: geometry collision cylinder length=0.043 radius=0.05; visual cylinder length=0.043 radius=0.05
- link right_front_wheel: geometry collision cylinder length=0.043 radius=0.05; visual cylinder length=0.043 radius=0.05

File: urdf/bvc.xacro (robot description, xacro)
@@ -9,5 +9,5 @@
   <xacro:wheel side="right" fob="back" sideDim="${rightWheelDist}" fobDim="${backWheelDist}" />
   <xacro:wheel side="left" fob="back" sideDim="${leftWheelDist}" fobDim="${backWheelDist}" />
-  <!-- <xacro:imu /> -->
+  <xacro:imu />
   <!-- <xacro:lidar /> TODO -->
     <xacro:include filename="$(find avc_urdf)/urdf/gazebo.xacro" />

File: urdf/geometries.xacro (robot description, xacro)
@@ -12,9 +12,9 @@
         </geometry>
 	</xacro:macro>
-    <!-- <xacro:macro name="imu_geometry">
+    <xacro:macro name="imu_geometry">
        <geometry>
             <box size = "${imuL} ${imuW} ${imuH} "/>
         </geometry>
-	</xacro:macro> -->
+	</xacro:macro>
     <xacro:macro name="wheel_mesh_geometry" params="side">
         <geometry>

File: urdf/inertial.xacro (robot description, xacro)
@@ -13,10 +13,10 @@
 		</inertial>
 	</xacro:macro>
-	<!-- <xacro:macro name="imu_inertial">
+	<xacro:macro name="imu_inertial">
 		<inertial>
             <mass value="${imuMass}"/>
             <inertia ixx="${imuIxx}" ixy="${imuIxy}" ixz="${imuIxz}" iyy="${imuIyy}" iyz="${imuIyz}" izz="${imuIzz}"/>
 		</inertial>
-	</xacro:macro> -->
+	</xacro:macro>
 	<xacro:macro name="axle_inertial">
 	    <inertial>

File: urdf/joints.xacro (robot description, xacro)
@@ -26,5 +26,5 @@
         </joint>
 	</xacro:macro>
-    <!-- <xacro:macro name="imu_joint">
+    <xacro:macro name="imu_joint">
         <joint name="imu_joint" type="fixed">
             <axis xyz="0 1 0"/>
@@ -33,5 +33,5 @@
             <origin xyz="0 0 0" />
         </joint>
-	</xacro:macro> -->
+	</xacro:macro>
     <xacro:macro name="chassis_box_joint">
         <joint name="chassis_box_joint" type="fixed">
@@ -39,5 +39,5 @@
             <parent link="base_link"/>
             <child link="chassis_box_link"/>
-            <origin xyz="0 0 0" />
+            <origin xyz="-.5 0 0" />
         </joint>
 	</xacro:macro>

File: urdf/links.xacro (robot description, xacro)
@@ -8,5 +8,6 @@
     <link name="base_link">
         <visual>
-            <xacro:chassis_mesh_geometry />
+            <!-- <xacro:chassis_mesh_geometry /> -->
+            <xacro:box_geometry />
         </visual>
         <collision>
@@ -19,5 +20,6 @@
     <link name="${side}_${fob}_wheel">
         <visual>
-            <xacro:wheel_mesh_geometry side="${side}"/>
+            <!-- <xacro:wheel_mesh_geometry side="${side}"/> -->
+            <xacro:wheel_geometry />
         </visual>
         <collision>
@@ -41,9 +43,9 @@
     <!-- <xacro:wheel_gazebo side="${side}" fob="${fob}"> -->
 </xacro:macro>
-<!-- <xacro:macro name="imu">
-    <link name="imu_link">
+<xacro:macro name="imu">
+    <link name="imu">
         <visual>
+            <!-- <xacro:imu_mesh_geometry /> -->
             <xacro:imu_geometry />
-            <material name="orange"/>
         </visual>
         <collision>
@@ -53,4 +55,4 @@
     </link>
     <xacro:imu_joint />
-</xacro:macro> -->
+</xacro:macro>
 </robot>

File: urdf/properties.xacro (robot description, xacro)
@@ -49,8 +49,10 @@
     <xacro:property name="wheelKd" value="1.0"/>
  <!-- ______________IMU parameters__________________________ -->
-    <!-- <xacro:property name="imuL" value="0.05" />
-    <xacro:property name="imuW" value="0.05" />
-    <xacro:property name="imuH" value="0.05" />
-    <xacro:property name="imuMass" value="10"/>
+    <xacro:property name="imuL" value="0.064" />
+    <xacro:property name="imuW" value="0.028" />
+    <xacro:property name="imuH" value="0.007" />
+imu
+imu
+    <xacro:property name="imuMass" value="0.1"/>
     <xacro:property name="imuIxx" value="0.4"/>
     <xacro:property name="imuIxy" value="0.4"/>
@@ -58,4 +60,8 @@
     <xacro:property name="imuIxz" value="0.4"/>
     <xacro:property name="imuIyz" value="0.4"/>
-    <xacro:property name="imuIzz" value="0.4"/> -->
+    <xacro:property name="imuIzz" value="0.4"/>
+     <!-- <xacro:property name="imuScale" value="0.001"/> -->
+    <xacro:property name="imuMeshXoffset" value="0.077"/>
+    <xacro:property name="imuMeshYoffset" value="0.070"/>
+    <xacro:property name="imuMeshZoffset" value="0.077"/>
 </robot>

File: urdf/transmissions.xacro (robot description, xacro)
@@ -23,3 +23,14 @@
         </transmission>
     </xacro:macro>
+    <xacro:macro name="imu_transmission" params="side fob">
+        <transmission name="${side}_${fob}_imu_trans">
+            <type>transmission_interface/SimpleTransmission</type>
+            <actuator name="${side}_${fob}_imu_motor">
+                <mechanicalReduction>1</mechanicalReduction>
+            </actuator>
+            <joint name="base_to_${side}_${fob}_imu">
+                <hardwareInterface>PositionJointInterface</hardwareInterface>
+            </joint>
+        </transmission>
+	</xacro:macro>
 </robot>
