Commit message: Dorky car

File: urdf/13-diffdrive.urdf.xacro (robot description, xacro)
@@ -1,4 +1,5 @@
 <?xml version="1.0"?>
-<robot name="roscontrol" xmlns:xacro="http://ros.org/wiki/xacro">
+<robot name="roscontrol"
+  xmlns:xacro="http://ros.org/wiki/xacro">
   <xacro:property name="width" value="0.2" />
   <xacro:property name="leglen" value="0.6" />
@@ -8,4 +9,7 @@
   <xacro:property name="wheeldiam" value="0.07" />
   <xacro:property name="pi" value="3.1415" />
+  <xacro:property name="chassisL" value="0.51" />
+  <xacro:property name="chassisW" value="0.2" />
+  <xacro:property name="chassisH" value="0.15" />
   <material name="blue">
     <color rgba="0 0 0.8 1"/>
@@ -26,5 +30,5 @@
     <visual>
       <geometry>
-        <cylinder radius="${width}" length="${bodylen}"/>
+        <box size = "${chassisL} ${chassisW} ${chassisH} "/>
       </geometry>
       <material name="blue"/>
@@ -32,10 +36,10 @@
     <collision>
       <geometry>
-        <cylinder radius="${width}" length="${bodylen}"/>
+        <box size = "${chassisL} ${chassisW} ${chassisH} "/>
       </geometry>
     </collision>
     <xacro:default_inertial mass="10"/>
   </link>
-  <xacro:macro name="wheel" params="prefix suffix reflect">
+  <xacro:macro name="wheel" params="prefix suffix reflect reflectL">
     <link name="${prefix}_${suffix}_wheel">
       <visual>
@@ -56,7 +60,7 @@
     <joint name="${prefix}_${suffix}_wheel_joint" type="continuous">
       <axis xyz="0 1 0" rpy="0 0 0" />
-      <parent link="${prefix}_base"/>
+      <parent link="base_link"/>
       <child link="${prefix}_${suffix}_wheel"/>
-      <origin xyz="${baselen*reflect/3} 0 -${wheeldiam/2+.05}" rpy="0 0 0"/>
+      <origin xyz="${baselen*reflect/3} ${baselen*reflectL} -${wheeldiam/2+.05}" rpy="0 0 0"/>
     </joint>
     <!-- This block provides the simulator (Gazebo) with information on a few additional
@@ -81,191 +85,8 @@
     </transmission>
   </xacro:macro>
-  <xacro:macro name="leg" params="prefix reflect">
-    <link name="${prefix}_leg">
-      <visual>
-        <geometry>
-          <box size="${leglen} 0.1 0.2"/>
-        </geometry>
-        <origin xyz="0 0 -${leglen/2}" rpy="0 ${pi/2} 0"/>
-        <material name="white"/>
-      </visual>
-      <collision>
-        <geometry>
-          <box size="${leglen} 0.1 0.2"/>
-        </geometry>
-        <origin xyz="0 0 -${leglen/2}" rpy="0 ${pi/2} 0"/>
-      </collision>
-      <xacro:default_inertial mass="10"/>
-    </link>
-    <joint name="base_to_${prefix}_leg" type="fixed">
-      <parent link="base_link"/>
-      <child link="${prefix}_leg"/>
-      <origin xyz="0 ${reflect*(width+.02)} 0.25" />
-    </joint>
-    <link name="${prefix}_base">
-      <visual>
-        <geometry>
-          <box size="${baselen} 0.1 0.1"/>
-        </geometry>
-        <material name="white"/>
-      </visual>
-      <collision>
-        <geometry>
-          <box size="${baselen} 0.1 0.1"/>
-        </geometry>
-      </collision>
-      <xacro:default_inertial mass="10"/>
-    </link>
-    <joint name="${prefix}_base_joint" type="fixed">
-      <parent link="${prefix}_leg"/>
-      <child link="${prefix}_base"/>
-      <origin xyz="0 0 ${-leglen}" />
-    </joint>
-    <xacro:wheel prefix="${prefix}" suffix="front" reflect="1"/>
-    <xacro:wheel prefix="${prefix}" suffix="back" reflect="-1"/>
-  </xacro:macro>
-  <xacro:leg prefix="right" reflect="-1" />
-  <xacro:leg prefix="left" reflect="1" />
-  <joint name="gripper_extension" type="prismatic">
-    <parent link="base_link"/>
-    <child link="gripper_pole"/>
-    <limit effort="1000.0" lower="-${width*2-.02}" upper="0" velocity="0.5"/>
-    <origin rpy="0 0 0" xyz="${width-.01} 0 0.2"/>
-    <limit effort="30" velocity="0.2"/>
-    <dynamics damping="0.0" friction="0.0"/>
-  </joint>
-  <link name="gripper_pole">
-    <visual>
-      <geometry>
-        <cylinder length="${polelen}" radius="0.01"/>
-      </geometry>
-      <origin xyz="${polelen/2} 0 0" rpy="0 ${pi/2} 0 "/>
-    </visual>
-    <collision>
-      <geometry>
-        <cylinder length="${polelen}" radius="0.01"/>
-      </geometry>
-      <origin xyz="${polelen/2} 0 0" rpy="0 ${pi/2} 0 "/>
-    </collision>
-    <xacro:default_inertial mass="0.05"/>
-  </link>
-  <transmission name="gripper_extension_trans">
-    <type>transmission_interface/SimpleTransmission</type>
-    <actuator name="gripper_extension_motor">
-      <mechanicalReduction>1</mechanicalReduction>
-    </actuator>
-    <joint name="gripper_extension">
-      <hardwareInterface>PositionJointInterface</hardwareInterface>
-    </joint>
-  </transmission>
-  <xacro:macro name="gripper" params="prefix reflect">
-    <joint name="${prefix}_gripper_joint" type="revolute">
-      <axis xyz="0 0 ${reflect}"/>
-      <limit effort="1000.0" lower="0.0" upper="0.548" velocity="0.5"/>
-      <origin rpy="0 0 0" xyz="${polelen} ${reflect*0.01} 0"/>
-      <parent link="gripper_pole"/>
-      <child link="${prefix}_gripper"/>
-      <limit effort="30" velocity="1.0"/>
-      <dynamics damping="0.0" friction="0.0"/>
-    </joint>
-    <link name="${prefix}_gripper">
-      <visual>
-        <origin rpy="${(reflect-1)/2*pi} 0 0" xyz="0 0 0"/>
-        <geometry>
-          <mesh filename="package://urdf_tutorial/meshes/l_finger.dae"/>
-        </geometry>
-      </visual>
-      <collision>
-        <geometry>
-          <mesh filename="package://urdf_tutorial/meshes/l_finger.dae"/>
-        </geometry>
-        <origin rpy="${(reflect-1)/2*pi} 0 0" xyz="0 0 0"/>
-      </collision>
-      <xacro:default_inertial mass="0.05"/>
-    </link>
-    <transmission name="${prefix}_gripper_trans">
-      <type>transmission_interface/SimpleTransmission</type>
-      <actuator name="${prefix}_gripper_motor">
-        <mechanicalReduction>1</mechanicalReduction>
-      </actuator>
-      <joint name="${prefix}_gripper_joint">
-        <hardwareInterface>PositionJointInterface</hardwareInterface>
-      </joint>
-    </transmission>
-    <joint name="${prefix}_tip_joint" type="fixed">
-      <parent link="${prefix}_gripper"/>
-      <child link="${prefix}_tip"/>
-    </joint>
-    <link name="${prefix}_tip">
-      <visual>
-        <origin rpy="${(reflect-1)/2*pi} 0 0" xyz="0.09137 0.00495 0"/>
-        <geometry>
-          <mesh filename="package://urdf_tutorial/meshes/l_finger_tip.dae"/>
-        </geometry>
-      </visual>
-      <collision>
-        <geometry>
-          <mesh filename="package://urdf_tutorial/meshes/l_finger_tip.dae"/>
-        </geometry>
-        <origin rpy="${(reflect-1)/2*pi} 0 0" xyz="0.09137 0.00495 0"/>
-      </collision>
-      <xacro:default_inertial mass="0.05"/>
-    </link>
-  </xacro:macro>
-  <xacro:gripper prefix="left" reflect="1" />
-  <xacro:gripper prefix="right" reflect="-1" />
-  <link name="head">
-    <visual>
-      <geometry>
-        <sphere radius="${width}"/>
-      </geometry>
-      <material name="white"/>
-    </visual>
-    <collision>
-      <geometry>
-        <sphere radius="${width}"/>
-      </geometry>
-    </collision>
-    <xacro:default_inertial mass="2"/>
-  </link>
-  <joint name="head_swivel" type="continuous">
-    <parent link="base_link"/>
-    <child link="head"/>
-    <axis xyz="0 0 1"/>
-    <origin xyz="0 0 ${bodylen/2}"/>
-    <limit effort="30" velocity="1.0"/>
-    <dynamics damping="0.0" friction="0.0"/>
-  </joint>
-  <!-- This block connects the head_swivel joint to an actuator (motor), which informs both
-  simulation and visualization of the robot -->
-  <transmission name="head_swivel_trans">
-    <type>transmission_interface/SimpleTransmission</type>
-    <actuator name="$head_swivel_motor">
-      <mechanicalReduction>1</mechanicalReduction>
-    </actuator>
-    <joint name="head_swivel">
-      <hardwareInterface>PositionJointInterface</hardwareInterface>
-    </joint>
-  </transmission>
-  <link name="box">
-    <visual>
-      <geometry>
-        <box size="0.08 0.08 0.08"/>
-      </geometry>
-      <material name="blue"/>
-      <origin xyz="-0.04 0 0"/>
-    </visual>
-    <collision>
-      <geometry>
-        <box size="0.08 0.08 0.08"/>
-      </geometry>
-    </collision>
-    <xacro:default_inertial mass="1"/>
-  </link>
-  <joint name="tobox" type="fixed">
-    <parent link="head"/>
-    <child link="box"/>
-    <origin xyz="${.707*width+0.04} 0 ${.707*width}"/>
-  </joint>
+    <xacro:wheel prefix="right" suffix="front" reflect="1" reflectL="1"/>
+    <xacro:wheel prefix="left" suffix="front" reflect="1" reflectL="-1"/>
+    <xacro:wheel prefix="right" suffix="back" reflect="-1" reflectL="1"/>
+    <xacro:wheel prefix="left" suffix="back" reflect="-1" reflectL="-1"/>
   <!-- Gazebo plugin for ROS Control -->
   <gazebo>

Commit message: Car moving with correct wheels

File: urdf/13-diffdrive.urdf.xacro (robot description, xacro)
@@ -12,4 +12,7 @@
   <xacro:property name="chassisW" value="0.2" />
   <xacro:property name="chassisH" value="0.15" />
+  <xacro:property name="seperationWheelDist" value=".1215" />
+  <xacro:property name="frontWheelDist" value="0.1535" />
+  <xacro:property name="backWheelDist" value="-0.1763" />
   <material name="blue">
     <color rgba="0 0 0.8 1"/>
@@ -41,5 +44,5 @@
     <xacro:default_inertial mass="10"/>
   </link>
-  <xacro:macro name="wheel" params="prefix suffix reflect reflectL">
+  <xacro:macro name="wheel" params="prefix suffix fb lr">
     <link name="${prefix}_${suffix}_wheel">
       <visual>
@@ -62,5 +65,5 @@
       <parent link="base_link"/>
       <child link="${prefix}_${suffix}_wheel"/>
-      <origin xyz="${baselen*reflect/3} ${baselen*reflectL} -${wheeldiam/2+.05}" rpy="0 0 0"/>
+      <origin xyz="${fb} ${lr} -${wheeldiam/2+.05}" rpy="0 0 0"/>
     </joint>
     <!-- This block provides the simulator (Gazebo) with information on a few additional
@@ -85,8 +88,8 @@
     </transmission>
   </xacro:macro>
-    <xacro:wheel prefix="right" suffix="front" reflect="1" reflectL="1"/>
-    <xacro:wheel prefix="left" suffix="front" reflect="1" reflectL="-1"/>
-    <xacro:wheel prefix="right" suffix="back" reflect="-1" reflectL="1"/>
-    <xacro:wheel prefix="left" suffix="back" reflect="-1" reflectL="-1"/>
+  <xacro:wheel prefix="right" suffix="front" fb="${frontWheelDist}" lr="${seperationWheelDist}"/>
+  <xacro:wheel prefix="left" suffix="front" fb="${frontWheelDist}" lr="${-seperationWheelDist}"/>
+  <xacro:wheel prefix="right" suffix="back" fb="${backWheelDist}" lr="${seperationWheelDist}"/>
+  <xacro:wheel prefix="left" suffix="back" fb="${backWheelDist}" lr="${-seperationWheelDist}"/>
   <!-- Gazebo plugin for ROS Control -->
   <gazebo>

Commit message: With Mesh

File: urdf/13-diffdrive.urdf.xacro (robot description, xacro)
@@ -15,4 +15,8 @@
   <xacro:property name="frontWheelDist" value="0.1535" />
   <xacro:property name="backWheelDist" value="-0.1763" />
+  <xacro:property name="chassisScale" value="0.001"/>
+  <xacro:property name="chassisMeshXoffset" value="-0.125"/>
+  <xacro:property name="chassisMeshYoffset" value="-0.070"/>
+  <xacro:property name="chassisMeshZoffset" value="-0.085"/>
   <material name="blue">
     <color rgba="0 0 0.8 1"/>
@@ -33,7 +37,7 @@
     <visual>
       <geometry>
-        <box size = "${chassisL} ${chassisW} ${chassisH} "/>
+        <mesh filename="file:///$(find avc_urdf)/meshes/chassis2.DAE" scale="${chassisScale} ${chassisScale} ${chassisScale}"/>
       </geometry>
-      <material name="blue"/>
+      <origin rpy="1.57 0 0" xyz="${chassisMeshXoffset} ${chassisMeshYoffset} ${chassisMeshZoffset}" />
     </visual>
     <collision>
@@ -88,8 +92,8 @@
     </transmission>
   </xacro:macro>
-  <xacro:wheel prefix="right" suffix="front" fb="${frontWheelDist}" lr="${seperationWheelDist}"/>
-  <xacro:wheel prefix="left" suffix="front" fb="${frontWheelDist}" lr="${-seperationWheelDist}"/>
-  <xacro:wheel prefix="right" suffix="back" fb="${backWheelDist}" lr="${seperationWheelDist}"/>
-  <xacro:wheel prefix="left" suffix="back" fb="${backWheelDist}" lr="${-seperationWheelDist}"/>
+  <xacro:wheel prefix="right" suffix="front" fb="${frontWheelDist}" lr="${-seperationWheelDist}"/>
+  <xacro:wheel prefix="left" suffix="front" fb="${frontWheelDist}" lr="${seperationWheelDist}"/>
+  <xacro:wheel prefix="right" suffix="back" fb="${backWheelDist}" lr="${-seperationWheelDist}"/>
+  <xacro:wheel prefix="left" suffix="back" fb="${backWheelDist}" lr="${seperationWheelDist}"/>
   <!-- Gazebo plugin for ROS Control -->
   <gazebo>

Commit message: Meshes

File: urdf/13-diffdrive.urdf.xacro (robot description, xacro)
@@ -9,9 +9,9 @@
   <xacro:property name="wheeldiam" value="0.07" />
   <xacro:property name="pi" value="3.1415" />
-  <xacro:property name="chassisL" value="0.51" />
+  <!-- <xacro:property name="chassisL" value="0.51" />
   <xacro:property name="chassisW" value="0.2" />
-  <xacro:property name="chassisH" value="0.15" />
+  <xacro:property name="chassisH" value="0.15" /> -->
   <xacro:property name="seperationWheelDist" value=".1215" />
-  <xacro:property name="frontWheelDist" value="0.1535" />
+  <!-- <xacro:property name="frontWheelDist" value="0.1535" />
   <xacro:property name="backWheelDist" value="-0.1763" />
   <xacro:property name="chassisScale" value="0.001"/>
@@ -19,4 +19,12 @@
   <xacro:property name="chassisMeshYoffset" value="-0.070"/>
   <xacro:property name="chassisMeshZoffset" value="-0.085"/>
+  <xacro:property name="wheelDrop" value="-0.075" />
+  <xacro:property name="wheelScale" value="0.001"/>
+  <xacro:property name="wheelMeshXoffset" value="0"/>
+  <xacro:property name="wheelMeshYoffset" value="0.022"/>
+  <xacro:property name="wheelMeshYoffsetLeft" value="-0.022"/>
+  <xacro:property name="wheelMeshZoffset" value="0"/> -->
+  <xacro:include filename="$(find avc_urdf)/urdf/properties.xacro" />
+  <xacro:include filename="$(find avc_urdf)/urdf/geometries.xacro" />
   <material name="blue">
     <color rgba="0 0 0.8 1"/>
@@ -51,15 +59,9 @@
     <link name="${prefix}_${suffix}_wheel">
       <visual>
-        <origin xyz="0 0 0" rpy="${pi/2} 0 0" />
-        <geometry>
-          <cylinder radius="${wheeldiam/2}" length="0.1"/>
-        </geometry>
-        <material name="black"/>
+        <xacro:wheel_mesh_geometry side="${prefix}"/>
+        <material name="black" />
       </visual>
       <collision>
-        <origin xyz="0 0 0" rpy="${pi/2} 0 0" />
-        <geometry>
-          <cylinder radius="${wheeldiam/2}" length="0.1"/>
-        </geometry>
+        <xacro:wheel_geometry />
       </collision>
       <xacro:default_inertial mass="1"/>
