Commit message: Fix Gazebo Materials

File: urdf/gazebo.xacro (robot description, xacro)
@@ -3,34 +3,32 @@
     <xacro:macro name="wheel_gazebo" params="prefix suffix">
         <gazebo reference="${prefix}_${suffix}_wheel">
-        <mu1 value="200.0"/>
-        <mu2 value="100.0"/>
-        <kp value="10000000.0" />
-        <kd value="1.0" />
-        <material>Gazebo/Grey</material>
+            <mu1 value="200.0"/>
+            <mu2 value="100.0"/>
+            <kp value="10000000.0" />
+            <kd value="1.0" />
+            <material>Gazebo/Grey</material>
         </gazebo>
     </xacro:macro>
-    <!-- <xacro:macro name="imu_gazebo">
-        <gazebo reference="imu">
-        <material>Gazebo/Red</material>
+    <xacro:macro name="imu_gazebo">
+        <gazebo reference="imu_link">
+            <material>Gazebo/Red</material>
         </gazebo>
     </xacro:macro>
     <xacro:macro name="lidar_gazebo">
-        <gazebo reference="lidar">
-        <visual>
-              <material>
-                <ambient>1.0 1.0 1.0 1.0</ambient>
-                <diffuse>1.0 1.0 1.0 1.0</diffuse>
-                <specular>1.0 1.0 1.0 1.0</specular>
-                <emissive>1.0 1.0 1.0 1.0</emissive>
-             </material>
-        </visual>
+        <gazebo reference="lidar_link">
+            <material>Gazebo/Blue</material>
         </gazebo>
-    </xacro:macro> -->
+    </xacro:macro>
+    <xacro:macro name="base_gazebo">
+        <gazebo reference="base_link">
+            <material>Gazebo/Black</material>
+        </gazebo>
+    </xacro:macro>
     <gazebo>
-		<plugin name="gazebo_ros_control" filename="libgazebo_ros_control.so">
-			<robotNamespace>/</robotNamespace>
-			<robotSimType>gazebo_ros_control/DefaultRobotHWSim</robotSimType>
+        <plugin name="gazebo_ros_control" filename="libgazebo_ros_control.so">
+            <robotNamespace>/</robotNamespace>
+            <robotSimType>gazebo_ros_control/DefaultRobotHWSim</robotSimType>
             <legacyModeNS>true</legacyModeNS>
-		</plugin>
-	</gazebo>
+        </plugin>
+    </gazebo>
 </robot>

File: urdf/links.xacro (robot description, xacro)
@@ -1,24 +1,25 @@
 <?xml version="1.0"?>
 <robot xmlns:xacro="http://www.ros.org/wiki/xacro" name="mintaur">
-	<xacro:include filename="$(find avc_urdf)/urdf/inertial.xacro" />
-	<xacro:include filename="$(find avc_urdf)/urdf/joints.xacro" />
-	<xacro:include filename="$(find avc_urdf)/urdf/transmissions.xacro" />
+  <xacro:include filename="$(find avc_urdf)/urdf/inertial.xacro" />
+  <xacro:include filename="$(find avc_urdf)/urdf/joints.xacro" />
+  <xacro:include filename="$(find avc_urdf)/urdf/transmissions.xacro" />
   <xacro:include filename="$(find avc_urdf)/urdf/geometries.xacro" />
-<xacro:macro name="base_link">
- <link name="base_link">
-    <visual>
-      <geometry>
-        <mesh filename="file:///$(find avc_urdf)/meshes/chassis2.DAE" scale="${chassisScale} ${chassisScale} ${chassisScale}"/>
-      </geometry>
-      <origin rpy="1.57 0 0" xyz="${chassisMeshXoffset} ${chassisMeshYoffset} ${chassisMeshZoffset}" />
-    </visual>
-    <collision>
-      <geometry>
-        <box size = "${chassisL} ${chassisW} ${chassisH} "/>
-      </geometry>
-    </collision>
-    <xacro:default_inertial mass="10"/>
-  </link>
-</xacro:macro>
+  <xacro:macro name="base_link">
+    <link name="base_link">
+      <visual>
+        <geometry>
+          <mesh filename="file:///$(find avc_urdf)/meshes/chassis2.DAE" scale="${chassisScale} ${chassisScale} ${chassisScale}"/>
+        </geometry>
+        <origin rpy="1.57 0 0" xyz="${chassisMeshXoffset} ${chassisMeshYoffset} ${chassisMeshZoffset}" />
+      </visual>
+      <collision>
+        <geometry>
+          <box size = "${chassisL} ${chassisW} ${chassisH} "/>
+        </geometry>
+      </collision>
+      <xacro:default_inertial mass="10"/>
+    </link>
+    <xacro:base_gazebo/>
+  </xacro:macro>
   <xacro:macro name="wheel" params="prefix suffix fb lr">
     <link name="${prefix}_${suffix}_wheel">
@@ -40,30 +41,30 @@
     <xacro:wheel_transmission prefix="${prefix}" suffix="${suffix}" />
   </xacro:macro>
-<xacro:macro name="imu">
+  <xacro:macro name="imu">
     <link name="imu_link">
-        <visual>
-            <xacro:imu_geometry />
-        </visual>
-        <collision>
-            <xacro:imu_geometry />
-        </collision>
-        <xacro:imu_inertial />
+      <visual>
+        <xacro:imu_geometry />
+      </visual>
+      <collision>
+        <xacro:imu_geometry />
+      </collision>
+      <xacro:imu_inertial />
     </link>
     <xacro:imu_joint />
-    <!-- <xacro:imu_gazebo /> -->
-</xacro:macro>
-<xacro:macro name="lidar">
+    <xacro:imu_gazebo />
+  </xacro:macro>
+  <xacro:macro name="lidar">
     <link name="lidar_link">
-        <visual>
-            <xacro:lidar_geometry />
-            <material name="blue" />
-        </visual>
-        <collision>
-            <xacro:lidar_geometry />
-        </collision>
-        <xacro:lidar_inertial />
+      <visual>
+        <xacro:lidar_geometry />
+        <material name="blue" />
+      </visual>
+      <collision>
+        <xacro:lidar_geometry />
+      </collision>
+      <xacro:lidar_inertial />
     </link>
     <xacro:lidar_joint />
-    <!-- <xacro:lidar_gazebo /> -->
-</xacro:macro>
+    <xacro:lidar_gazebo />
+  </xacro:macro>
 </robot>
