Commit message: Now bvc has movement

File: urdf/bvc.xacro (robot description, xacro)
@@ -6,8 +6,8 @@
     <xacro:include filename="$(find avc_urdf)/urdf/gazebo.xacro" />
   <xacro:base_link/>
-  <xacro:wheel side="right" fob="front" sideDim="${rightWheelDist}" fobDim="${frontWheelDist}" />
-  <xacro:wheel side="left" fob="front" sideDim="${leftWheelDist}" fobDim="${frontWheelDist}" />
-  <xacro:wheel side="right" fob="back" sideDim="${rightWheelDist}" fobDim="${backWheelDist}" />
-  <xacro:wheel side="left" fob="back" sideDim="${leftWheelDist}" fobDim="${backWheelDist}" />
+  <xacro:wheel prefix="right" suffix="front" fb="${frontWheelDist}" lr="${-seperationWheelDist}"/>
+  <xacro:wheel prefix="left" suffix="front" fb="${frontWheelDist}" lr="${seperationWheelDist}"/>
+  <xacro:wheel prefix="right" suffix="back" fb="${backWheelDist}" lr="${-seperationWheelDist}"/>
+  <xacro:wheel prefix="left" suffix="back" fb="${backWheelDist}" lr="${seperationWheelDist}"/>
   <!-- <xacro:imu /> -->
   <!-- <xacro:lidar /> TODO -->

File: urdf/inertial.xacro (robot description, xacro)
@@ -7,8 +7,14 @@
 		</inertial>
 	</xacro:macro>
+	<xacro:macro name="default_inertial" params="mass">
+		<inertial>
+			<mass value="${mass}" />
+			<inertia ixx="1.0" ixy="0.0" ixz="0.0" iyy="1.0" iyz="0.0" izz="1.0" />
+		</inertial>
+	</xacro:macro>
 	<xacro:macro name="wheel_inertial">
 		<inertial>
-            <mass value="${wheelMass}"/>
-            <inertia ixx="${wheelIxx}" ixy="${wheelIxy}" ixz="${wheelIxz}" iyy="${wheelIyy}" iyz="${wheelIyz}" izz="${wheelIzz}"/>
+			<mass value="${wheelMass}"/>
+			<inertia ixx="${wheelIxx}" ixy="${wheelIxy}" ixz="${wheelIxz}" iyy="${wheelIyy}" iyz="${wheelIyz}" izz="${wheelIzz}"/>
 		</inertial>
 	</xacro:macro>
@@ -20,8 +26,8 @@
 	</xacro:macro> -->
 	<xacro:macro name="axle_inertial">
-	    <inertial>
-            <mass value="0.001"/>
-            <inertia ixx="0.0" ixy="0.0" ixz="0.0" iyy="0.0" iyz="0.0" izz="0.0"/>
-        </inertial>
+		<inertial>
+			<mass value="0.001"/>
+			<inertia ixx="0.0" ixy="0.0" ixz="0.0" iyy="0.0" iyz="0.0" izz="0.0"/>
+		</inertial>
 	</xacro:macro>
 </robot>

File: urdf/links.xacro (robot description, xacro)
@@ -6,41 +6,57 @@
     <xacro:include filename="$(find avc_urdf)/urdf/geometries.xacro" />
 <xacro:macro name="base_link">
-    <link name="base_link">
-        <visual>
-            <xacro:chassis_mesh_geometry />
-            <material name="white" />
-        </visual>
-        <collision>
-            <xacro:box_geometry />
-        </collision>
-        <xacro:box_inertial />
+ <link name="base_link">
+    <visual>
+      <geometry>
+        <mesh filename="file:///$(find avc_urdf)/meshes/chassis2.DAE" scale="${chassisScale} ${chassisScale} ${chassisScale}"/>
+      </geometry>
+      <origin rpy="1.57 0 0" xyz="${chassisMeshXoffset} ${chassisMeshYoffset} ${chassisMeshZoffset}" />
+    </visual>
+    <collision>
+      <geometry>
+        <box size = "${chassisL} ${chassisW} ${chassisH} "/>
+      </geometry>
+    </collision>
+    <xacro:default_inertial mass="10"/>
+  </link>
+</xacro:macro>
+  <xacro:macro name="wheel" params="prefix suffix fb lr">
+    <link name="${prefix}_${suffix}_wheel">
+      <visual>
+        <xacro:wheel_mesh_geometry side="${prefix}"/>
+        <material name="black" />
+      </visual>
+      <collision>
+        <xacro:wheel_geometry />
+      </collision>
+      <xacro:default_inertial mass="1"/>
     </link>
-</xacro:macro>
-<xacro:macro name="wheel" params="side fob sideDim fobDim">
-    <link name="${side}_${fob}_wheel">
-        <visual>
-            <xacro:wheel_mesh_geometry side="${side}"/>
-            <material name="black" />
-        </visual>
-        <collision>
-            <xacro:wheel_geometry />
-        </collision>
-        <xacro:wheel_inertial />
-    </link>
-    <!-- Use this block for a front wheel -->
-    <xacro:if value="${fob =='front'}">
-        <link name="${side}_${fob}_axle">
-            <xacro:axle_inertial />
-        </link>
-        <xacro:axle_joint side="${side}" fob="${fob}" sideDim="${sideDim}" fobDim="${fobDim}"/>
-        <xacro:front_wheel_joint side="${side}" fob="${fob}" sideDim="${sideDim}" fobDim="${fobDim}"/>
-        <xacro:axle_transmission side="${side}" fob="${fob}"/>
-    </xacro:if>
-    <!-- Use this block for a rear wheel -->
-    <xacro:if value="${fob =='back'}">
-        <xacro:rear_wheel_joint side="${side}" fob="${fob}" sideDim="${sideDim}" fobDim="${fobDim}"/>
-    </xacro:if>
-    <xacro:wheel_gazebo side="${side}" fob="${fob}"/>
-</xacro:macro>
+    <joint name="${prefix}_${suffix}_wheel_joint" type="continuous">
+      <axis xyz="0 1 0" rpy="0 0 0" />
+      <parent link="base_link"/>
+      <child link="${prefix}_${suffix}_wheel"/>
+      <origin xyz="${fb} ${lr} -${wheeldiam/2+.05}" rpy="0 0 0"/>
+    </joint>
+    <!-- This block provides the simulator (Gazebo) with information on a few additional
+    physical properties. See http://gazebosim.org/tutorials/?tut=ros_urdf for more-->
+    <gazebo reference="${prefix}_${suffix}_wheel">
+      <mu1 value="200.0"/>
+      <mu2 value="100.0"/>
+      <kp value="10000000.0" />
+      <kd value="1.0" />
+      <material>Gazebo/Grey</material>
+    </gazebo>
+    <!-- This block connects the wheel joint to an actuator (motor), which informs both
+    simulation and visualization of the robot -->
+    <transmission name="${prefix}_${suffix}_wheel_trans">
+      <type>transmission_interface/SimpleTransmission</type>
+      <actuator name="${prefix}_${suffix}_wheel_motor">
+        <mechanicalReduction>1</mechanicalReduction>
+      </actuator>
+      <joint name="${prefix}_${suffix}_wheel_joint">
+        <hardwareInterface>VelocityJointInterface</hardwareInterface>
+      </joint>
+    </transmission>
+  </xacro:macro>
 <!-- <xacro:macro name="imu">
     <link name="imu_link">

File: urdf/properties.xacro (robot description, xacro)
@@ -1,6 +1,6 @@
 <?xml version="1.0"?>
 <robot xmlns:xacro="http://www.ros.org/wiki/xacro" name="mintaur">
-	<!-- X axis direction is forward, Y axis direction is left -->
- <!-- ______________Chassis parameters__________________________ -->
+    <!-- X axis direction is forward, Y axis direction is left -->
+    <!-- ______________Chassis parameters__________________________ -->
     <xacro:property name="chassisL" value="0.51" />
     <xacro:property name="chassisW" value="0.2" />
@@ -13,9 +13,9 @@
     <xacro:property name="chassisIyz" value="0.0"/>
     <xacro:property name="chassisIzz" value="0.0"/>
-     <xacro:property name="chassisScale" value="0.001"/>
+    <xacro:property name="chassisScale" value="0.001"/>
     <xacro:property name="chassisMeshXoffset" value="-0.125"/>
     <xacro:property name="chassisMeshYoffset" value="-0.070"/>
     <xacro:property name="chassisMeshZoffset" value="-0.085"/>
- <!-- ______________Wheel parameters__________________________ -->
+    <!-- ______________Wheel parameters__________________________ -->
     <!-- Wheel Rotation Limits> -->
     <xacro:property name="llimit" value="-0.785" />
@@ -30,5 +30,5 @@
     <xacro:property name="wheelMeshXoffset" value="0"/>
     <xacro:property name="wheelMeshYoffset" value="0.022"/>
-   <xacro:property name="wheelMeshYoffsetLeft" value="-0.022"/>
+    <xacro:property name="wheelMeshYoffsetLeft" value="-0.022"/>
     <xacro:property name="wheelMeshZoffset" value="0"/>
     <!-- Wheel Physical Propreties-->
@@ -49,5 +49,5 @@
     <xacro:property name="wheelKp" value="10000000.0"/>
     <xacro:property name="wheelKd" value="1.0"/>
- <!-- ______________IMU parameters__________________________ -->
+    <!-- ______________IMU parameters__________________________ -->
     <!-- <xacro:property name="imuL" value="0.05" />
     <xacro:property name="imuW" value="0.05" />
@@ -60,3 +60,11 @@
     <xacro:property name="imuIyz" value="0.4"/>
     <xacro:property name="imuIzz" value="0.4"/> -->
+    <xacro:property name="width" value="0.2" />
+    <xacro:property name="leglen" value="0.6" />
+    <xacro:property name="polelen" value="0.2" />
+    <xacro:property name="bodylen" value="0.6" />
+    <xacro:property name="baselen" value="0.4" />
+    <xacro:property name="wheeldiam" value="0.07" />
+    <xacro:property name="pi" value="3.1415" />
+    <xacro:property name="seperationWheelDist" value=".1215" />
 </robot>

Commit message: Laser geometries

File: urdf/bvc.xacro (robot description, xacro)
@@ -11,4 +11,4 @@
   <xacro:wheel side="left" fob="back" sideDim="${leftWheelDist}" fobDim="${backWheelDist}" />
   <!-- <xacro:imu /> -->
-  <!-- <xacro:lidar /> TODO -->
+  <xacro:lidar />
 </robot>

File: urdf/geometries.xacro (robot description, xacro)
@@ -3,5 +3,5 @@
     <xacro:macro name="chassis_mesh_geometry">
         <geometry>
-            <mesh filename="file:///$(find avc_urdf)/meshes/chassis2.DAE" scale="${chassisScale} ${chassisScale} ${chassisScale}"/>
+            <mesh filename='file://$(find avc_urdf)/meshes/chassis2.DAE' scale="${chassisScale} ${chassisScale} ${chassisScale}"/>
          </geometry>
          <origin rpy="1.57 0 0" xyz="${chassisMeshXoffset} ${chassisMeshYoffset} ${chassisMeshZoffset}" />
@@ -19,5 +19,5 @@
     <xacro:macro name="wheel_mesh_geometry" params="side">
         <geometry>
-            <mesh filename="file:///$(find avc_urdf)/meshes/wheels.DAE" scale="${wheelScale} ${wheelScale} ${wheelScale}"/>
+            <mesh filename='file://$(find avc_urdf)/meshes/wheels.DAE' scale="${wheelScale} ${wheelScale} ${wheelScale}"/>
          </geometry>
             <xacro:if value="${side =='right'}">
@@ -34,3 +34,9 @@
         <origin rpy="1.57075 0 0" xyz="0 0 0"/>
 	</xacro:macro>
+    <xacro:macro name="lidar_geometry">
+        <geometry>
+            <cylinder length="${lidarThick}" radius="${lidarRadius}"/>
+        </geometry>
+        <origin rpy="0 0 0" xyz="0 0 0"/>
+	</xacro:macro>
 </robot>

File: urdf/inertial.xacro (robot description, xacro)
@@ -9,6 +9,6 @@
 	<xacro:macro name="wheel_inertial">
 		<inertial>
-            <mass value="${wheelMass}"/>
-            <inertia ixx="${wheelIxx}" ixy="${wheelIxy}" ixz="${wheelIxz}" iyy="${wheelIyy}" iyz="${wheelIyz}" izz="${wheelIzz}"/>
+            	<mass value="${wheelMass}"/>
+            	<inertia ixx="${wheelIxx}" ixy="${wheelIxy}" ixz="${wheelIxz}" iyy="${wheelIyy}" iyz="${wheelIyz}" izz="${wheelIzz}"/>
 		</inertial>
 	</xacro:macro>
@@ -25,3 +25,9 @@
         </inertial>
 	</xacro:macro>
+	<xacro:macro name="lidar_inertial">
+		<inertial>
+            	<mass value="${lidarMass}"/>
+            	<inertia ixx="${lidarIxx}" ixy="${lidarIxy}" ixz="${lidarIxz}" iyy="${lidarIyy}" iyz="${lidarIyz}" izz="${lidarIzz}"/>
+		</inertial>
+	</xacro:macro>
 </robot>

File: urdf/joints.xacro (robot description, xacro)
@@ -42,3 +42,11 @@
         </joint>
 	</xacro:macro>
+    <xacro:macro name="lidar_joint">
+        <joint name="lidar_joint" type="fixed">
+            <parent link="base_link"/>
+            <child link="lidar_link"/>
+            <origin xyz="0.076 0.0 0.059"/>
+            <!-- <origin xyz="0 0 0"/> -->
+        </joint>
+    </xacro:macro>
 </robot>

File: urdf/links.xacro (robot description, xacro)
@@ -56,3 +56,17 @@
     <xacro:imu_joint />
 </xacro:macro> -->
+<xacro:macro name="lidar">
+    <link name="lidar_link">
+        <visual>
+            <xacro:lidar_geometry />
+            <!-- <xacro:chassis_mesh_geometry /> -->
+            <material name="grey" />
+        </visual>
+        <collision>
+            <xacro:lidar_geometry />
+        </collision>
+        <xacro:lidar_inertial />
+    </link>
+    <xacro:lidar_joint />
+</xacro:macro>
 </robot>

File: urdf/properties.xacro (robot description, xacro)
@@ -60,3 +60,13 @@
     <xacro:property name="imuIyz" value="0.4"/>
     <xacro:property name="imuIzz" value="0.4"/> -->
+ <!-- ______________Lidar parameters__________________________ -->
+    <xacro:property name="lidarThick" value="0.086" />
+    <xacro:property name="lidarRadius" value="0.045" />
+    <xacro:property name="lidarMass" value="0.025"/>
+    <xacro:property name="lidarIxx" value="0.08333333*lidarMass*((3*(lidarRadius*lidarRadius))+(lidarThick*lidarThick))"/>
+    <xacro:property name="lidarIxy" value="0.0"/>
+    <xacro:property name="lidarIyy" value="0.08333333*lidarMass*((3*(lidarRadius*lidarRadius))+(lidarThick*lidarThick))"/>
+    <xacro:property name="lidarIxz" value="0.0"/>
+    <xacro:property name="lidarIyz" value="0.0"/>
+    <xacro:property name="lidarIzz" value="0.5*lidarMass*(lidarRadius*lidarRadius)"/>
 </robot>
