Commit message: Merge Lidar and IMU. Need Colors

File: urdf/bvc.xacro (robot description, xacro)
@@ -10,5 +10,5 @@
   <xacro:wheel prefix="right" suffix="back" fb="${backWheelDist}" lr="${-seperationWheelDist}"/>
   <xacro:wheel prefix="left" suffix="back" fb="${backWheelDist}" lr="${seperationWheelDist}"/>
-  <!-- <xacro:imu /> -->
-  <!-- <xacro:lidar /> TODO -->
+  <xacro:imu />
+  <xacro:lidar />
 </robot>

File: urdf/gazebo.xacro (robot description, xacro)
@@ -1,13 +1,30 @@
 <?xml version="1.0"?>
 <robot xmlns:xacro="http://www.ros.org/wiki/xacro" name="mintaur">
-    <xacro:macro name="wheel_gazebo" params="side fob">
-        <gazebo reference="${side}_${fob}_wheel">
-            <mu1 value="${wheelMu1}"/>
-            <mu2 value="{wheelMu2}"/>
-            <kp value="{wheelKp}" />
-            <kd value="{wheelKd}" />
-            <material>Gazebo/Grey</material>
+    <xacro:macro name="wheel_gazebo" params="prefix suffix">
+        <gazebo reference="${prefix}_${suffix}_wheel">
+        <mu1 value="200.0"/>
+        <mu2 value="100.0"/>
+        <kp value="10000000.0" />
+        <kd value="1.0" />
+        <material>Gazebo/Grey</material>
         </gazebo>
     </xacro:macro>
+    <!-- <xacro:macro name="imu_gazebo">
+        <gazebo reference="imu">
+        <material>Gazebo/Red</material>
+        </gazebo>
+    </xacro:macro>
+    <xacro:macro name="lidar_gazebo">
+        <gazebo reference="lidar">
+        <visual>
+              <material>
+                <ambient>1.0 1.0 1.0 1.0</ambient>
+                <diffuse>1.0 1.0 1.0 1.0</diffuse>
+                <specular>1.0 1.0 1.0 1.0</specular>
+                <emissive>1.0 1.0 1.0 1.0</emissive>
+             </material>
+        </visual>
+        </gazebo>
+    </xacro:macro> -->
     <gazebo>
 		<plugin name="gazebo_ros_control" filename="libgazebo_ros_control.so">

File: urdf/geometries.xacro (robot description, xacro)
@@ -34,3 +34,14 @@
         <origin rpy="1.57075 0 0" xyz="0 0 0"/>
 	</xacro:macro>
+   <xacro:macro name="imu_geometry">
+       <geometry>
+            <box size = "${imuL} ${imuW} ${imuH} "/>
+        </geometry>
+    </xacro:macro>
+    <xacro:macro name="lidar_geometry">
+        <geometry>
+            <cylinder length="${lidarThick}" radius="${lidarRadius}"/>
+        </geometry>
+        <origin rpy="0 0 0" xyz="0 0 0"/>
+    </xacro:macro>
 </robot>

File: urdf/inertial.xacro (robot description, xacro)
@@ -19,10 +19,4 @@
 		</inertial>
 	</xacro:macro>
-	<!-- <xacro:macro name="imu_inertial">
-		<inertial>
-            <mass value="${imuMass}"/>
-            <inertia ixx="${imuIxx}" ixy="${imuIxy}" ixz="${imuIxz}" iyy="${imuIyy}" iyz="${imuIyz}" izz="${imuIzz}"/>
-		</inertial>
-	</xacro:macro> -->
 	<xacro:macro name="axle_inertial">
 		<inertial>
@@ -31,3 +25,15 @@
 		</inertial>
 	</xacro:macro>
+	<xacro:macro name="imu_inertial">
+		<inertial>
+            <mass value="${imuMass}"/>
+            <inertia ixx="${imuIxx}" ixy="${imuIxy}" ixz="${imuIxz}" iyy="${imuIyy}" iyz="${imuIyz}" izz="${imuIzz}"/>
+		</inertial>
+	</xacro:macro>
+	<xacro:macro name="lidar_inertial">
+		<inertial>
+            	<mass value="${lidarMass}"/>
+            	<inertia ixx="${lidarIxx}" ixy="${lidarIxy}" ixz="${lidarIxz}" iyy="${lidarIyy}" iyz="${lidarIyz}" izz="${lidarIzz}"/>
+		</inertial>
+	</xacro:macro>
 </robot>

File: urdf/joints.xacro (robot description, xacro)
@@ -1,4 +1,12 @@
 <?xml version="1.0"?>
 <robot xmlns:xacro="http://www.ros.org/wiki/xacro" name="mintaur">
+	<xacro:macro name="wheel_move_joint" params="prefix suffix fb lr">
+        <joint name="${prefix}_${suffix}_wheel_joint" type="continuous">
+        <axis xyz="0 1 0" rpy="0 0 0" />
+        <parent link="base_link"/>
+        <child link="${prefix}_${suffix}_wheel"/>
+        <origin xyz="${fb} ${lr} ${-wheeldiam/2-.05}" rpy="0 0 0"/>
+        </joint>
+	</xacro:macro>
 	<xacro:macro name="axle_joint" params="side fob sideDim fobDim">
         <joint name="base_to_${side}_${fob}_axle" type="revolute">
@@ -26,12 +34,4 @@
         </joint>
 	</xacro:macro>
-    <!-- <xacro:macro name="imu_joint">
-        <joint name="imu_joint" type="fixed">
-            <axis xyz="0 1 0"/>
-            <parent link="base_link"/>
-            <child link="imu_link"/>
-            <origin xyz="0 0 0" />
-        </joint>
-	</xacro:macro> -->
     <xacro:macro name="chassis_box_joint">
         <joint name="chassis_box_joint" type="fixed">
@@ -42,3 +42,18 @@
         </joint>
 	</xacro:macro>
+    <xacro:macro name="imu_joint">
+        <joint name="imu_joint" type="fixed">
+            <axis xyz="0 1 0"/>
+            <parent link="base_link"/>
+            <child link="imu_link"/>
+            <origin xyz="${imuXoffset} ${imuYoffset} ${imuZoffset}" />
+        </joint>
+    </xacro:macro>
+    <xacro:macro name="lidar_joint">
+        <joint name="lidar_joints" type="fixed">
+            <parent link="base_link"/>
+            <child link="lidar_link"/>
+            <origin xyz="${lidarXoffset} ${lidarYoffset} ${lidarZoffset}"/>
+        </joint>
+    </xacro:macro>
 </robot>

File: urdf/links.xacro (robot description, xacro)
@@ -4,5 +4,5 @@
 	<xacro:include filename="$(find avc_urdf)/urdf/joints.xacro" />
 	<xacro:include filename="$(find avc_urdf)/urdf/transmissions.xacro" />
-    <xacro:include filename="$(find avc_urdf)/urdf/geometries.xacro" />
+  <xacro:include filename="$(find avc_urdf)/urdf/geometries.xacro" />
 <xacro:macro name="base_link">
  <link name="base_link">
@@ -30,38 +30,18 @@
         <xacro:wheel_geometry />
       </collision>
-      <xacro:default_inertial mass="1"/>
+      <xacro:wheel_inertial />
     </link>
-    <joint name="${prefix}_${suffix}_wheel_joint" type="continuous">
-      <axis xyz="0 1 0" rpy="0 0 0" />
-      <parent link="base_link"/>
-      <child link="${prefix}_${suffix}_wheel"/>
-      <origin xyz="${fb} ${lr} -${wheeldiam/2+.05}" rpy="0 0 0"/>
-    </joint>
+    <xacro:wheel_move_joint prefix="${prefix}" suffix="${suffix}" fb="${fb}" lr="${lr}" />
     <!-- This block provides the simulator (Gazebo) with information on a few additional
     physical properties. See http://gazebosim.org/tutorials/?tut=ros_urdf for more-->
-    <gazebo reference="${prefix}_${suffix}_wheel">
-      <mu1 value="200.0"/>
-      <mu2 value="100.0"/>
-      <kp value="10000000.0" />
-      <kd value="1.0" />
-      <material>Gazebo/Grey</material>
-    </gazebo>
+    <xacro:wheel_gazebo prefix="${prefix}" suffix="${suffix}" />
     <!-- This block connects the wheel joint to an actuator (motor), which informs both
     simulation and visualization of the robot -->
-    <transmission name="${prefix}_${suffix}_wheel_trans">
-      <type>transmission_interface/SimpleTransmission</type>
-      <actuator name="${prefix}_${suffix}_wheel_motor">
-        <mechanicalReduction>1</mechanicalReduction>
-      </actuator>
-      <joint name="${prefix}_${suffix}_wheel_joint">
-        <hardwareInterface>VelocityJointInterface</hardwareInterface>
-      </joint>
-    </transmission>
+    <xacro:wheel_transmission prefix="${prefix}" suffix="${suffix}" />
   </xacro:macro>
-<!-- <xacro:macro name="imu">
+<xacro:macro name="imu">
     <link name="imu_link">
         <visual>
             <xacro:imu_geometry />
-            <material name="orange"/>
         </visual>
         <collision>
@@ -71,4 +51,19 @@
     </link>
     <xacro:imu_joint />
-</xacro:macro> -->
+    <!-- <xacro:imu_gazebo /> -->
+</xacro:macro>
+<xacro:macro name="lidar">
+    <link name="lidar_link">
+        <visual>
+            <xacro:lidar_geometry />
+            <material name="blue" />
+        </visual>
+        <collision>
+            <xacro:lidar_geometry />
+        </collision>
+        <xacro:lidar_inertial />
+    </link>
+    <xacro:lidar_joint />
+    <!-- <xacro:lidar_gazebo /> -->
+</xacro:macro>
 </robot>

File: urdf/properties.xacro (robot description, xacro)
@@ -49,9 +49,9 @@
     <xacro:property name="wheelKp" value="10000000.0"/>
     <xacro:property name="wheelKd" value="1.0"/>
-    <!-- ______________IMU parameters__________________________ -->
-    <!-- <xacro:property name="imuL" value="0.05" />
-    <xacro:property name="imuW" value="0.05" />
-    <xacro:property name="imuH" value="0.05" />
-    <xacro:property name="imuMass" value="10"/>
+ <!-- ______________IMU parameters__________________________ -->
+    <xacro:property name="imuL" value="0.064" />
+    <xacro:property name="imuW" value="0.028" />
+    <xacro:property name="imuH" value="0.007" />
+    <xacro:property name="imuMass" value="0.1"/>
     <xacro:property name="imuIxx" value="0.4"/>
     <xacro:property name="imuIxy" value="0.4"/>
@@ -59,5 +59,9 @@
     <xacro:property name="imuIxz" value="0.4"/>
     <xacro:property name="imuIyz" value="0.4"/>
-    <xacro:property name="imuIzz" value="0.4"/> -->
+    <xacro:property name="imuIzz" value="0.4"/>
+    <xacro:property name="imuXoffset" value="-0.077"/>
+    <xacro:property name="imuYoffset" value="0.0"/>
+    <xacro:property name="imuZoffset" value="0.077"/>
+<!-- __________________Random Values______________________ -->
     <xacro:property name="width" value="0.2" />
     <xacro:property name="leglen" value="0.6" />
@@ -68,3 +72,16 @@
     <xacro:property name="pi" value="3.1415" />
     <xacro:property name="seperationWheelDist" value=".1215" />
+     <!-- ______________Lidar parameters__________________________ -->
+    <xacro:property name="lidarThick" value="0.086" />
+    <xacro:property name="lidarRadius" value="0.045" />
+    <xacro:property name="lidarXoffset" value="0.076"/>
+    <xacro:property name="lidarYoffset" value="0.0"/>
+    <xacro:property name="lidarZoffset" value="0.059"/>
+    <xacro:property name="lidarMass" value="0.025"/>
+    <xacro:property name="lidarIxx" value="${0.08333333*lidarMass*(3*lidarRadius*lidarRadius+lidarThick*lidarThick)}"/>
+    <xacro:property name="lidarIxy" value="0.0"/>
+    <xacro:property name="lidarIyy" value="${0.08333333*lidarMass*(3*lidarRadius*lidarRadius+lidarThick*lidarThick)}"/>
+    <xacro:property name="lidarIxz" value="0.0"/>
+    <xacro:property name="lidarIyz" value="0.0"/>
+    <xacro:property name="lidarIzz" value="${0.5*lidarMass*(lidarRadius*lidarRadius)}"/>
 </robot>

File: urdf/transmissions.xacro (robot description, xacro)
@@ -13,11 +13,11 @@
         </transmission>
 	</xacro:macro>
-    <xacro:macro name="wheel_transmission" params="side fob">
-        <transmission name="${side}_${fob}_wheel_trans">
+    <xacro:macro name="wheel_transmission" params="prefix suffix">
+        <transmission name="${prefix}_${suffix}_wheel_trans">
             <type>transmission_interface/SimpleTransmission</type>
-            <actuator name="${side}_${fob}_wheel_motor">
+            <actuator name="${prefix}_${suffix}_wheel_motor">
                 <mechanicalReduction>1</mechanicalReduction>
             </actuator>
-            <joint name="${side}_${fob}_wheel_joint">
+            <joint name="${prefix}_${suffix}_wheel_joint">
                 <hardwareInterface>hardware_interface/VelocityJointInterface</hardwareInterface>
             </joint>

Commit message: Reformat

File: urdf/bvc.xacro (robot description, xacro)
@@ -2,13 +2,13 @@
 <robot xmlns:xacro="http://www.ros.org/wiki/xacro" name="mintaur">
     <xacro:include filename="$(find avc_urdf)/urdf/materials.xacro" />
-	<xacro:include filename="$(find avc_urdf)/urdf/properties.xacro" />
+    <xacro:include filename="$(find avc_urdf)/urdf/properties.xacro" />
     <xacro:include filename="$(find avc_urdf)/urdf/links.xacro" />
     <xacro:include filename="$(find avc_urdf)/urdf/gazebo.xacro" />
-  <xacro:base_link/>
-  <xacro:wheel prefix="right" suffix="front" fb="${frontWheelDist}" lr="${-seperationWheelDist}"/>
-  <xacro:wheel prefix="left" suffix="front" fb="${frontWheelDist}" lr="${seperationWheelDist}"/>
-  <xacro:wheel prefix="right" suffix="back" fb="${backWheelDist}" lr="${-seperationWheelDist}"/>
-  <xacro:wheel prefix="left" suffix="back" fb="${backWheelDist}" lr="${seperationWheelDist}"/>
-  <xacro:imu />
-  <xacro:lidar />
+    <xacro:base_link/>
+    <xacro:wheel prefix="right" suffix="front" fb="${frontWheelDist}" lr="${-seperationWheelDist}"/>
+    <xacro:wheel prefix="left" suffix="front" fb="${frontWheelDist}" lr="${seperationWheelDist}"/>
+    <xacro:wheel prefix="right" suffix="back" fb="${backWheelDist}" lr="${-seperationWheelDist}"/>
+    <xacro:wheel prefix="left" suffix="back" fb="${backWheelDist}" lr="${seperationWheelDist}"/>
+    <xacro:imu />
+    <xacro:lidar />
 </robot>

File: urdf/inertial.xacro (robot description, xacro)
@@ -27,12 +27,12 @@
 	<xacro:macro name="imu_inertial">
 		<inertial>
-            <mass value="${imuMass}"/>
-            <inertia ixx="${imuIxx}" ixy="${imuIxy}" ixz="${imuIxz}" iyy="${imuIyy}" iyz="${imuIyz}" izz="${imuIzz}"/>
+			<mass value="${imuMass}"/>
+			<inertia ixx="${imuIxx}" ixy="${imuIxy}" ixz="${imuIxz}" iyy="${imuIyy}" iyz="${imuIyz}" izz="${imuIzz}"/>
 		</inertial>
 	</xacro:macro>
 	<xacro:macro name="lidar_inertial">
 		<inertial>
-            	<mass value="${lidarMass}"/>
-            	<inertia ixx="${lidarIxx}" ixy="${lidarIxy}" ixz="${lidarIxz}" iyy="${lidarIyy}" iyz="${lidarIyz}" izz="${lidarIzz}"/>
+			<mass value="${lidarMass}"/>
+			<inertia ixx="${lidarIxx}" ixy="${lidarIxy}" ixz="${lidarIxz}" iyy="${lidarIyy}" iyz="${lidarIyz}" izz="${lidarIzz}"/>
 		</inertial>
 	</xacro:macro>

File: urdf/materials.xacro (robot description, xacro)
@@ -1,30 +1,31 @@
 <?xml version="1.0"?>
-<robot name="mintaur" xmlns:xacro="http://www.ros.org/wiki/xacro">
+<robot name="mintaur"
+    xmlns:xacro="http://www.ros.org/wiki/xacro">
     <material name="black">
-    <color rgba="0.0 0.0 0.0 1.0"/>
+        <color rgba="0.0 0.0 0.0 1.0"/>
     </material>
     <material name="blue">
-    <color rgba="0.0 0.0 0.8 1.0"/>
+        <color rgba="0.0 0.0 0.8 1.0"/>
     </material>
     <material name="green">
-    <color rgba="0.0 0.8 0.0 1.0"/>
+        <color rgba="0.0 0.8 0.0 1.0"/>
     </material>
     <material name="grey">
-    <color rgba="0.2 0.2 0.2 1.0"/>
+        <color rgba="0.2 0.2 0.2 1.0"/>
     </material>
     <material name="orange">
-    <color rgba="${255/255} ${108/255} ${10/255} 1.0"/>
+        <color rgba="${255/255} ${108/255} ${10/255} 1.0"/>
     </material>
     <material name="brown">
-    <color rgba="${222/255} ${207/255} ${195/255} 1.0"/>
+        <color rgba="${222/255} ${207/255} ${195/255} 1.0"/>
     </material>
     <material name="red">
-    <color rgba="0.8 0.0 0.0 1.0"/>
+        <color rgba="0.8 0.0 0.0 1.0"/>
     </material>
     <material name="white">
-    <color rgba="1.0 1.0 1.0 1.0"/>
+        <color rgba="1.0 1.0 1.0 1.0"/>
     </material>
     <material name="acrylic">
-    <color rgba="1.0 1.0 1.0 0.4"/>
+        <color rgba="1.0 1.0 1.0 0.4"/>
     </material>
 </robot>

File: urdf/properties.xacro (robot description, xacro)
@@ -49,5 +49,5 @@
     <xacro:property name="wheelKp" value="10000000.0"/>
     <xacro:property name="wheelKd" value="1.0"/>
- <!-- ______________IMU parameters__________________________ -->
+    <!-- ______________IMU parameters__________________________ -->
     <xacro:property name="imuL" value="0.064" />
     <xacro:property name="imuW" value="0.028" />
@@ -63,5 +63,5 @@
     <xacro:property name="imuYoffset" value="0.0"/>
     <xacro:property name="imuZoffset" value="0.077"/>
-<!-- __________________Random Values______________________ -->
+    <!-- __________________Random Values______________________ -->
     <xacro:property name="width" value="0.2" />
     <xacro:property name="leglen" value="0.6" />
@@ -72,5 +72,5 @@
     <xacro:property name="pi" value="3.1415" />
     <xacro:property name="seperationWheelDist" value=".1215" />
-     <!-- ______________Lidar parameters__________________________ -->
+    <!-- ______________Lidar parameters__________________________ -->
     <xacro:property name="lidarThick" value="0.086" />
     <xacro:property name="lidarRadius" value="0.045" />

File: urdf/transmissions.xacro (robot description, xacro)
@@ -1,5 +1,6 @@
 <?xml version="1.0"?>
-<robot name="mintaur" xmlns:xacro="http://www.ros.org/wiki/xacro">
-	<xacro:macro name="axle_transmission" params="side fob">
+<robot name="mintaur"
+    xmlns:xacro="http://www.ros.org/wiki/xacro">
+    <xacro:macro name="axle_transmission" params="side fob">
         <transmission name="${side}_${fob}_axle_trans">
             <type>transmission_interface/SimpleTransmission</type>
@@ -12,5 +13,5 @@
             </joint>
         </transmission>
-	</xacro:macro>
+    </xacro:macro>
     <xacro:macro name="wheel_transmission" params="prefix suffix">
         <transmission name="${prefix}_${suffix}_wheel_trans">
