Commit message: Update mesh, Attempt Motion

File: avc_urdf/urdf/joints.xacro (robot description, xacro)
@@ -3,4 +3,12 @@
 	<xacro:macro name="wheel_move_joint" params="prefix suffix fb lr">
         <joint name="${prefix}_${suffix}_wheel_joint" type="continuous">
+        <axis xyz="0 1 0" rpy="0 0 0" />
+        <parent link="base_link"/>
+        <child link="${prefix}_${suffix}_wheel"/>
+        <origin xyz="${fb} ${lr} ${-wheeldiam/2-.05}" rpy="0 0 0"/>
+        </joint>
+	</xacro:macro>
+    <xacro:macro name="wheel_move_joint2" params="prefix suffix fb lr">
+        <joint name="$wheel_{prefix}_joint" type="continuous">
         <axis xyz="0 1 0" rpy="0 0 0" />
         <parent link="base_link"/>

File: avc_urdf/urdf/links.xacro (robot description, xacro)
@@ -18,5 +18,5 @@
         </geometry>
       </collision>
-      <xacro:default_inertial mass="10"/>
+      <!-- <xacro:default_inertial mass="10"/> -->
     </link>
     <xacro:base_gazebo/>

Commit message: Give wheels axels

File: avc_urdf/urdf/joints.xacro (robot description, xacro)
@@ -4,7 +4,7 @@
         <joint name="${prefix}_${suffix}_wheel_joint" type="continuous">
         <axis xyz="0 1 0" rpy="0 0 0" />
-        <parent link="base_link"/>
+        <parent link="${prefix}_${suffix}_axle"/>
         <child link="${prefix}_${suffix}_wheel"/>
-        <origin xyz="${fb} ${lr} ${-wheeldiam/2-.05}" rpy="0 0 0"/>
+        <origin xyz="0 0 0" rpy="0 0 0"/>
         </joint>
 	</xacro:macro>
@@ -17,11 +17,11 @@
         </joint>
 	</xacro:macro>
-	<xacro:macro name="axle_joint" params="side fob sideDim fobDim">
-        <joint name="base_to_${side}_${fob}_axle" type="revolute">
+	<xacro:macro name="axle_joint" params="prefix suffix fb lr">
+        <joint name="${prefix}_${suffix}_axle" type="revolute">
             <axis xyz="0 0 1"/>
             <limit effort="${axleEffort}" lower="${llimit}" upper="${ulimit}" velocity="${axleVelocity}"/>
             <parent link="base_link"/>
-            <child link="${side}_${fob}_axle"/>
-            <origin xyz="${fobDim} ${sideDim} ${wheelDrop}" />
+            <child link="${prefix}_${suffix}_axle"/>
+            <origin xyz="${fb} ${lr} ${wheelDrop}" />
         </joint>
 	</xacro:macro>

File: avc_urdf/urdf/links.xacro (robot description, xacro)
@@ -39,4 +39,6 @@
       <xacro:wheel_inertial />
     </link>
+    <link name="${prefix}_${suffix}_axle"/>
+  	<xacro:axle_joint prefix="${prefix}" suffix="${suffix}" fb="${fb}" lr="${lr}"/>
     <xacro:wheel_move_joint prefix="${prefix}" suffix="${suffix}" fb="${fb}" lr="${lr}" />
     <!-- This block provides the simulator (Gazebo) with information on a few additional

Commit message: Two wheel

File: avc_urdf/urdf/joints.xacro (robot description, xacro)
@@ -18,5 +18,5 @@
 	</xacro:macro>
 	<xacro:macro name="axle_joint" params="prefix suffix fb lr">
-        <joint name="${prefix}_${suffix}_axle" type="revolute">
+        <joint name="${prefix}_${suffix}_axle_joint" type="revolute">
             <axis xyz="0 0 1"/>
             <limit effort="${axleEffort}" lower="${llimit}" upper="${ulimit}" velocity="${axleVelocity}"/>
