Commit message: Movement with avc and wheels

File: avc_urdf/urdf/links.xacro (robot description, xacro)
@@ -6,4 +6,10 @@
   <xacro:include filename="$(find avc_urdf)/urdf/geometries.xacro" />
   <xacro:macro name="base_link">
+   <link name="base_footprint"/>
+  <joint name="base_joint" type="fixed">
+    <parent link="base_footprint"/>
+    <child link="base_link" />
+    <origin xyz="0 0 0.13" rpy="0 0 0"/>
+  </joint>
     <link name="base_link">
       <visual>

Commit message: In the right frame

File: avc_urdf/urdf/links.xacro (robot description, xacro)
@@ -10,5 +10,5 @@
     <parent link="base_footprint"/>
     <child link="base_link" />
-    <origin xyz="0 0 0.13" rpy="0 0 0"/>
+    <origin xyz="${-backWheelDist} 0 0.13" rpy="0 0 0"/>
   </joint>
     <link name="base_link">
