Commit message: Update Controller

File: avc_urdf/urdf/properties.xacro (robot description, xacro)
@@ -70,5 +70,5 @@
     <xacro:property name="baselen" value="0.4" />
     <xacro:property name="wheeldiam" value="0.07" />
-    <xacro:property name="pi" value="3.1415" />
+    <xacro:property name="pis" value="3.1415" />
     <xacro:property name="seperationWheelDist" value=".1215" />
     <!-- ______________Lidar parameters__________________________ -->
